File: microcontroller.kicad_sch (KiCad schematic)
At the start: 7 parts

Commit message: rearrange and connect everything
rearrange and connect everything
Connections:
- net GPIO_AUX: now also E1.5 (D35), R8.1; no longer E1.2 (VP), R3.1
- net I2C_SCL: now also E1.11 (D14); no longer E1.29 (D22)
- net I2C_SDA: now also E1.13 (D13); no longer E1.26 (D21)
- net LASER_PWM: now also E1.18 (D15); no longer E1.7 (D33)
- net MOT_EN: now also E1.20 (D4); no longer E1.18 (D15)
- net SD_CS: now also E1.29 (D22); no longer E1.23 (D5)
- net X_CS: now also E1.10 (D27); no longer E1.13 (D13)
- net X_DIR: now also E1.12 (D12); no longer E1.11 (D14)
- net X_LIMIT: now also E1.2 (VP), R3.1; no longer E1.4 (D34), R7.1
- net Y_CS: now also E1.8 (D25); no longer E1.10 (D27)
- net Y_DIR: now also E1.9 (D26); no longer E1.8 (D25)
- net Y_LIMIT: now also E1.4 (D34), R7.1; no longer E1.5 (D35), R8.1
- net Y_STEP: now also E1.23 (D5); no longer E1.9 (D26)
- net Z_CS: now also E1.6 (D32); no longer E1.20 (D4)
- net Z_DIR: now also E1.7 (D33); no longer E1.6 (D32)
- net Z_STEP: now also E1.26 (D21); no longer E1.12 (D12)
