File: power_delivery.kicad_sch (KiCad schematic)
At the start: 10 parts, among them J1 24v (motors), J2 24v (laser), J3 24v (everything else)

Commit message: rearrange and connect everything
rearrange and connect everything
Parts:
- J1: value 24v (motors) -> Motor Power
- J2: value 24v (laser) -> Laser Power
- J3: value 24v (everything else) -> System Power
Connections:
- net +24V_LASER renamed +LASER_PWR
- net +24V_MOTORS renamed +MOTOR_PWR
Changed lines of the file:
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@@
 		)
 	)
-	(global_label "+24V_MOTORS"
+	(global_label "+MOTOR_PWR"
 		(shape input)
 		(at 156.21 39.37 0)
@@
 		)
 	)
-	(global_label "+24V_LASER"
+	(global_label "+LASER_PWR"
 		(shape input)
 		(at 156.21 87.63 0)
@@
 			)
 		)
-		(property "Value" "24v (motors)"
+		(property "Value" "Motor Power"
 			(at 48.26 45.466 0)
 			(effects
@@
 			)
 		)
-		(property "Value" "24v (laser)"
+		(property "Value" "Laser Power"
 			(at 48.26 93.726 0)
 			(effects
@@
 			)
 		)
-		(property "Value" "24v (everything else)"
+		(property "Value" "System Power"
 			(at 48.26 147.32 0)
 			(effects
